File: cad_files/connecting/connecting.sch (KiCad schematic (older format))
At the start: 58 parts, among them M1 Motor_AC, M2 Motor_AC, M3 Motor_AC, M4 Motor_AC, P1 CONN_01X03, P1 SCREW_CONN_1, P13 SCREW_CONN_1, P14 SCREW_CONN_1, P15 SCREW_CONN_1, P16 SCREW_CONN_1, P17 SCREW_CONN_1, P18 SCREW_CONN_1, P19 SCREW_CONN_1, P2 SCREW_CONN_1, P20 SCREW_CONN_1, P21 SCREW_CONN_1, P22 SCREW_CONN_1, P23 SCREW_CONN_1, P24 SCREW_CONN_1, P25 SCREW_CONN_1, P26 SCREW_CONN_1, P27 SCREW_CONN_1, P28 SCREW_CONN_1, P29 SCREW_CONN_1, P3 SCREW_CONN_1, P30 SCREW_CONN_1, P31 SCREW_CONN_1, P32 SCREW_CONN_1, P33 SCREW_CONN_1, P34 SCREW_CONN_1, P4 SCREW_CONN_1, P5 SCREW_CONN_1, P6 SCREW_CONN_1, P7 SCREW_CONN_1, P8 SCREW_CONN_1, P9 SCREW_CONN_1, SW1 SWITCH_2P, SW2 SWITCH_2P, SW3 SWITCH_2P

Commit message: 190909
Parts:
- added F1: 16A, symbol Fuse
- renumbered La2 to La1, La3 to La2, La4 to La3, La5 to La4, La1 to La5, SW2 to SW1, SW3 to SW2, SW1 to SW3, P1 to X1
Connections:
- wire segments 177 -> 178
Changed lines of the file:
@@
 encoding utf-8
 Sheet 1 1
-Title "Connecting of device"
+Title "MM4A Electrical distribution and switching unit"
 Date "2019-09-19"
 Rev "190919"
 Comp "Pozsar Zsolt"
-Comment1 ""
+Comment1 "Connecting of unit"
 Comment2 ""
 Comment3 ""
@@
 $EndComp
 Text Notes 1500 1700 0    70   ~ 0
-230V\n50/60Hz
+  230V\n50/60Hz
 Text Notes 1325 1200 0    118  ~ 24
 MM4A
@@
 $EndComp
 $Comp
-L Lamp La1
+L Lamp La5
 U 1 1 5D7386FE
 P 2500 4600
-F 0 "La1" V 2825 4600 50  0000 C CNN
+F 0 "La5" V 2825 4600 50  0000 C CNN
 F 1 "230V" H 2650 4450 50  0001 C CNN
 F 2 "lamp" H 2700 4750 50  0001 C CNN
@@
 $EndComp
 $Comp
-L Lamp La2
+L Lamp La1
 U 1 1 5D7387FE
 P 9300 3700
-F 0 "La2" V 9125 3550 50  0000 C CNN
+F 0 "La1" V 9125 3550 50  0000 C CNN
 F 1 "230V" H 9450 3550 50  0001 C CNN
 F 2 "lamp" H 9500 3850 50  0001 C CNN
@@
 $EndComp
 $Comp
-L SWITCH_2P SW1
+L SWITCH_2P SW3
 U 1 1 5D7344B3
 P 2475 4000
-F 0 "SW1" V 2875 4300 50  0000 C CNN
+F 0 "SW3" V 2875 4300 50  0000 C CNN
 F 1 "SWITCH_2P" H 2525 3325 70  0001 C CNN
 F 2 "" H 2475 3850 60  0000 C CNN
@@
 PE
 $Comp
-L SWITCH_2P SW2
+L SWITCH_2P SW1
 U 1 1 5D736C18
 P 6625 4025
-F 0 "SW2" V 6275 3725 50  0000 C CNN
+F 0 "SW1" V 6275 3725 50  0000 C CNN
 F 1 "SWITCH_2P" H 6625 3775 70  0001 C CNN
 F 2 "" H 6625 3875 60  0000 C CNN
@@
 $EndComp
 $Comp
-L SWITCH_2P SW3
+L SWITCH_2P SW2
 U 1 1 5D7370EE
 P 7525 4025
-F 0 "SW3" V 7175 3725 50  0000 C CNN
+F 0 "SW2" V 7175 3725 50  0000 C CNN
 F 1 "SWITCH_2P" V 7525 3775 70  0001 C CNN
 F 2 "" H 7525 3875 60  0000 C CNN
@@
 NoConn ~ 2500 4700
 $Comp
-L Lamp La3
+L Lamp La2
 U 1 1 5D738E8B
 P 9300 4350
-F 0 "La3" V 9125 4200 50  0000 C CNN
+F 0 "La2" V 9125 4200 50  0000 C CNN
 F 1 "230V" H 9450 4200 50  0001 C CNN
 F 2 "lamp" H 9500 4500 50  0001 C CNN
@@
 $EndComp
 $Comp
-L Lamp La4
+L Lamp La3
 U 1 1 5D738F45
 P 9300 5000
-F 0 "La4" V 9150 4850 50  0000 C CNN
+F 0 "La3" V 9150 4850 50  0000 C CNN
 F 1 "230V" V 9450 4850 50  0001 C CNN
 F 2 "lamp" H 9500 5150 50  0001 C CNN
@@
 $EndComp
 $Comp
-L Lamp La5
+L Lamp La4
 U 1 1 5D739000
 P 9300 5650
-F 0 "La5" V 9150 5500 50  0000 C CNN
+F 0 "La4" V 9150 5500 50  0000 C CNN
 F 1 "230V" H 9450 5500 50  0001 C CNN
 F 2 "lamp" H 9500 5800 50  0001 C CNN
@@
 Connection ~ 7425 5200
 Wire Wire Line
-	1475 2300 1475 7025
+	1475 2300 1475 6525
+Wire Wire Line
+	1475 6825 1475 7025
 Wire Wire Line
 	1725 2300 1725 7025
@@
 	5600 3550 5600 2300
 $Comp
-L CONN_01X03 P1
+L CONN_01X03 X1
 U 1 1 5D744E76
 P 3525 4025
-F 0 "P1" V 3125 4300 50  0000 C CNN
+F 0 "X1" V 3125 4300 50  0000 C CNN
 F 1 "CONN_01X03" V 3625 4025 50  0001 C CNN
 F 2 "" H 3525 4025 50  0000 C CNN
@@
 Text Notes 3300 4225 0    60   ~ 0
 230V 10A
+$Comp
+L Fuse F1
+U 1 1 5D76B8DA
+P 1475 6675
+F 0 "F1" H 1575 6575 50  0000 C CNN
+F 1 "16A" H 1350 6775 50  0000 C CNN
+F 2 "" V 1405 6675 50  0000 C CNN
+F 3 "" H 1475 6675 50  0000 C CNN
+	1    1475 6675
+	-1   0    0    1
+$EndComp
 $EndSCHEMATC
