File: cad_files/mm4a/mm4a.sch (KiCad schematic (older format))
At the start: 68 parts, among them K1 Electromagnetic_Actor, K1a SWITCH_1P, K1b SWITCH_1P, K2 Electromagnetic_Actor, K2a SWITCH_1P, K2b SWITCH_1P, K3 Electromagnetic_Actor, K3a SWITCH_1P, K3b SWITCH_1P, K4 Electromagnetic_Actor, K4a SWITCH_1P, K4b SWITCH_1P, K5 Electromagnetic_Actor, K5a SWITCH_1P, K5b SWITCH_1P, P1 SCREW_CONN_1, P10 SCREW_CONN_1, P11 SCREW_CONN_1, P12 SCREW_CONN_1, P13 SCREW_CONN_1, P14 SCREW_CONN_1, P15 SCREW_CONN_1, P16 SCREW_CONN_1, P17 SCREW_CONN_1, P18 SCREW_CONN_1, P19 SCREW_CONN_1, P2 SCREW_CONN_1, P20 SCREW_CONN_1, P21 SCREW_CONN_1, P22 SCREW_CONN_1, P23 SCREW_CONN_1, P24 SCREW_CONN_1, P25 SCREW_CONN_1, P26 SCREW_CONN_1, P27 SCREW_CONN_1, P28 SCREW_CONN_1, P29 SCREW_CONN_1, P3 SCREW_CONN_1, P30 SCREW_CONN_1, P31 SCREW_CONN_1, P32 SCREW_CONN_1, P33 SCREW_CONN_1, P34 SCREW_CONN_1, P4 SCREW_CONN_1, P5 SCREW_CONN_1, P6 SCREW_CONN_1, P7 SCREW_CONN_1, P8 SCREW_CONN_1, P9 SCREW_CONN_1, SW1 SWITCH_2P

Commit message: 190909
Parts:
- F7: value 3A -> 2A
- renumbered F5 to F4, F6 to F5, F7 to F6
Connections:
- new net: F1.~ (B), F2.~ (B), F3.~ (B), F4.~ (B), F5.~ (B), F6.~ (B), F7.1, La1.1 (-), SW1.2
Other:
- moved on the sheet: K1a, K1b, K2a, K2b, K3a, K3b
Changed lines of the file:
@@
 encoding utf-8
 Sheet 1 1
-Title "MM4A Growing house controlling equipment"
+Title "MM4A Electrical distribution and switching unit"
 Date "2019-09-19"
 Rev "190919"
@@
 $EndComp
 $Comp
-L Overcurrent_breaker F5
+L Overcurrent_breaker F4
 U 1 1 5CA26594
 P 8300 2650
-F 0 "F5" V 8150 2750 50  0000 C CNN
+F 0 "F4" V 8150 2750 50  0000 C CNN
 F 1 "C10A" V 8150 2525 50  0000 C CNN
 F 2 "~" H 8325 2650 50  0001 C CNN
@@
 U 1 1 5CA2659A
 P 8300 3700
-F 0 "K1a" V 8150 3800 50  0000 C CNN
+F 0 "K1a" V 8520 3800 50  0000 C CNN
 F 1 "SWITCH_1P" H 8300 3600 70  0001 C CNN
 F 2 "~" H 8300 3700 60  0000 C CNN
 F 3 "~" H 8300 3700 60  0000 C CNN
 	1    8300 3700
-	0    -1   -1   0
-$EndComp
-$Comp
-L Overcurrent_breaker F6
+	0    1    -1   0
+$EndComp
+$Comp
+L Overcurrent_breaker F5
 U 1 1 5CA39A8A
 P 9250 2650
-F 0 "F6" V 9100 2750 50  0000 C CNN
+F 0 "F5" V 9100 2750 50  0000 C CNN
 F 1 "B6A" V 9100 2550 50  0000 C CNN
 F 2 "~" H 9275 2650 50  0001 C CNN
@@
 F 3 "~" H 9250 4000 60  0000 C CNN
 	1    9250 4000
-	0    -1   -1   0
-$EndComp
-$Comp
-L Overcurrent_breaker F7
+	0    1    -1   0
+$EndComp
+$Comp
+L Overcurrent_breaker F6
 U 1 1 5CA3A398
 P 10200 2650
-F 0 "F7" V 10050 2750 50  0000 C CNN
+F 0 "F6" V 10050 2750 50  0000 C CNN
 F 1 "C6A" V 10050 2550 50  0000 C CNN
 F 2 "~" H 10225 2650 50  0001 C CNN
@@
 F 3 "~" H 10200 4200 60  0000 C CNN
 	1    10200 4200
-	0    -1   -1   0
+	0    1    -1   0
 $EndComp
 $Comp
@@
 U 1 1 5D72D25F
 P 8550 3700
-F 0 "K1b" V 8400 3800 50  0000 C CNN
+F 0 "K1b" V 8770 3810 50  0000 C CNN
 F 1 "SWITCH_1P" H 8550 3600 70  0001 C CNN
 F 2 "~" H 8550 3700 60  0000 C CNN
 F 3 "~" H 8550 3700 60  0000 C CNN
 	1    8550 3700
-	0    -1   -1   0
+	0    1    -1   0
 $EndComp
 $Comp
@@
 F 3 "~" H 9500 4000 60  0000 C CNN
 	1    9500 4000
-	0    -1   -1   0
+	0    1    -1   0
 $EndComp
 $Comp
@@
 F 3 "~" H 10450 4200 60  0000 C CNN
 	1    10450 4200
-	0    -1   -1   0
+	0    1    -1   0
 $EndComp
 $Comp
@@
 P 4050 2550
 F 0 "F7" H 4200 2650 50  0000 C CNN
-F 1 "3A" H 3925 2450 50  0000 C CNN
+F 1 "2A" H 3925 2450 50  0000 C CNN
 F 2 "" V 3980 2550 50  0000 C CNN
 F 3 "" H 4050 2550 50  0000 C CNN
@@
 Connection ~ 3300 1800
 Wire Notes Line
-	7950 4200 10150 4200
+	7950 4200 10500 4200
 Wire Notes Line
-	9200 4000 7000 4000
+	7000 4000 9550 4000
 Wire Notes Line
-	8250 3700 6050 3700
+	6050 3700 8600 3700
 Wire Wire Line
 	4350 1600 4350 1550
